Commit message: wip fixing joint names

File: robots/descriptions/go2_description/xacro/gazebo.xacro (robot description, xacro)
@@ -92,9 +92,9 @@
     </gazebo> -->
     <!-- FL leg -->
-    <gazebo reference="lf_hip_link">
+    <gazebo reference="FL_hip">
         <mu1>0.2</mu1>
         <mu2>0.2</mu2>
     </gazebo>
-    <gazebo reference="lf_upper_leg_link">
+    <gazebo reference="FL_thigh">
         <mu1>0.2</mu1>
         <mu2>0.2</mu2>
@@ -103,10 +103,10 @@
         <kd>1.0</kd>
     </gazebo>
-    <gazebo reference="lf_lower_leg_link">
+    <gazebo reference="FL_calf">
         <mu1>0.2</mu1>
         <mu2>0.2</mu2>
         <self_collide>1</self_collide>
     </gazebo>
-    <gazebo reference="lf_foot_link">
+    <gazebo reference="FL_foot">
         <mu1>0.6</mu1>
         <mu2>0.6</mu2>
@@ -116,9 +116,9 @@
     </gazebo>
     <!-- FR leg -->
-    <gazebo reference="rf_hip">
+    <gazebo reference="FR_hip">
         <mu1>0.2</mu1>
         <mu2>0.2</mu2>
     </gazebo>
-    <gazebo reference="rf_upper_leg_link">
+    <gazebo reference="FR_thigh">
         <mu1>0.2</mu1>
         <mu2>0.2</mu2>
@@ -127,10 +127,10 @@
         <kd>1.0</kd>
     </gazebo>
-    <gazebo reference="rf_lower_leg_link">
+    <gazebo reference="FR_calf">
         <mu1>0.2</mu1>
         <mu2>0.2</mu2>
         <self_collide>1</self_collide>
     </gazebo>
-    <gazebo reference="rf_foot_link">
+    <gazebo reference="FR_foot">
         <mu1>0.6</mu1>
         <mu2>0.6</mu2>
@@ -140,9 +140,9 @@
     </gazebo>
     <!-- RL leg -->
-    <gazebo reference="lh_hip">
+    <gazebo reference="RL_hip">
         <mu1>0.2</mu1>
         <mu2>0.2</mu2>
     </gazebo>
-    <gazebo reference="lh_upper_leg_link">
+    <gazebo reference="RL_thigh">
         <mu1>0.2</mu1>
         <mu2>0.2</mu2>
@@ -151,10 +151,10 @@
         <kd>1.0</kd>
     </gazebo>
-    <gazebo reference="lh_lower_leg_link">
+    <gazebo reference="RL_calf">
         <mu1>0.2</mu1>
         <mu2>0.2</mu2>
         <self_collide>1</self_collide>
     </gazebo>
-    <gazebo reference="lh_foot_link">
+    <gazebo reference="RL_foot">
         <mu1>0.6</mu1>
         <mu2>0.6</mu2>
@@ -164,9 +164,9 @@
     </gazebo>
     <!-- RR leg -->
-    <gazebo reference="rh_hip">
+    <gazebo reference="RR_hip">
         <mu1>0.2</mu1>
         <mu2>0.2</mu2>
     </gazebo>
-    <gazebo reference="rh_upper_leg_link">
+    <gazebo reference="RR_thigh">
         <mu1>0.2</mu1>
         <mu2>0.2</mu2>
@@ -175,10 +175,10 @@
         <kd>1.0</kd>
     </gazebo>
-    <gazebo reference="rh_lower_leg_link">
+    <gazebo reference="RR_calf">
         <mu1>0.2</mu1>
         <mu2>0.2</mu2>
         <self_collide>1</self_collide>
     </gazebo>
-    <gazebo reference="rh_foot_link">
+    <gazebo reference="RR_foot">
         <mu1>0.6</mu1>
         <mu2>0.6</mu2>

File: robots/descriptions/go2_description/xacro/leg.xacro (robot description, xacro)
@@ -17,5 +17,5 @@
             </xacro:if>
             <parent link="trunk"/>
-            <child link="${name}_hip_link"/>
+            <child link="${name}_hip"/>
             <axis xyz="1 0 0"/>
             <dynamics damping="${damping}" friction="${friction}"/>
@@ -27,5 +27,5 @@
             </xacro:if>
         </joint>
-        <link name="${name}_hip_link">
+        <link name="${name}_hip">
             <visual>
                 <xacro:if value="${(mirror_dae == True) and (front_hind_dae == True)}">
@@ -61,13 +61,13 @@
             </inertial>
         </link>
-        <joint name="${name}_upper_leg_joint" type="revolute">
+        <joint name="${name}_thigh_joint" type="revolute">
             <origin rpy="0 0 0" xyz="0 ${thigh_offset*mirror} 0"/>
-            <parent link="${name}_hip_link"/>
-            <child link="${name}_upper_leg_link"/>
+            <parent link="${name}_hip"/>
+            <child link="${name}_thigh"/>
             <axis xyz="0 1 0"/>
             <dynamics damping="${damping}" friction="${friction}"/>
             <limit effort="${thigh_torque_max}" velocity="${thigh_velocity_max}" lower="${thigh_position_min}" upper="${thigh_position_max}"/>
         </joint>
-        <link name="${name}_upper_leg_link">
+        <link name="${name}_thigh">
             <visual>
                 <origin rpy="0 0 0" xyz="0 0 0"/>
@@ -97,13 +97,13 @@
             </inertial>
         </link>
-        <joint name="${name}_lower_leg_joint" type="revolute">
+        <joint name="${name}_calf_joint" type="revolute">
             <origin rpy="0 0 0" xyz="0 0 ${-thigh_length}"/>
-            <parent link="${name}_upper_leg_link"/>
-            <child link="${name}_lower_leg_link"/>
+            <parent link="${name}_thigh"/>
+            <child link="${name}_calf"/>
             <axis xyz="0 1 0"/>
             <dynamics damping="${damping}" friction="${friction}"/>
             <limit effort="${calf_torque_max}" velocity="${calf_velocity_max}" lower="${calf_position_min}" upper="${calf_position_max}"/>
         </joint>
-        <link name="${name}_lower_leg_link">
+        <link name="${name}_calf">
             <visual>
                 <origin rpy="0 0 0" xyz="0 0 0"/>
@@ -130,8 +130,8 @@
         <joint name="${name}_foot_joint" type="fixed">0
             <origin rpy="0 0 0" xyz="0 0 ${-(calf_length)}"/>
-            <parent link="${name}_lower_leg_link"/>
-            <child link="${name}_foot_link"/>
+            <parent link="${name}_calf"/>
+            <child link="${name}_foot"/>
         </joint>
-        <link name="${name}_foot_link">
+        <link name="${name}_foot">
             <visual>
                 <origin rpy="0 0 0" xyz="0 0 0"/>
@@ -164,10 +164,10 @@
                 <state_interface name="velocity"/>
             </joint>
-            <joint name="${name}_upper_leg_joint">
+            <joint name="${name}_thigh_joint">
                 <command_interface name="effort"/>
                 <state_interface name="position"/>
                 <state_interface name="velocity"/>
             </joint>
-            <joint name="${name}_lower_leg_joint">
+            <joint name="${name}_calf_joint">
                 <command_interface name="effort"/>
                 <state_interface name="position"/>

File: robots/descriptions/go2_description/xacro/robot.xacro (robot description, xacro)
@@ -106,7 +106,7 @@
     </link>
 -->
-    <xacro:leg name="rf" mirror="-1" mirror_dae= "False" front_hind="1"  front_hind_dae="True"  />
-    <xacro:leg name="lf" mirror="1"  mirror_dae="True"   front_hind="1"  front_hind_dae="True"  />
-    <xacro:leg name="rh" mirror="-1" mirror_dae="False"  front_hind="-1" front_hind_dae="False" />
-    <xacro:leg name="lh" mirror="1"  mirror_dae="True"   front_hind="-1" front_hind_dae="False" />
+    <xacro:leg name="FL" mirror="1"  mirror_dae="True"   front_hind="1"  front_hind_dae="True"  />
+    <xacro:leg name="FR" mirror="-1" mirror_dae= "False" front_hind="1"  front_hind_dae="True"  />
+    <xacro:leg name="RL" mirror="1"  mirror_dae="True"   front_hind="-1" front_hind_dae="False" />
+    <xacro:leg name="RR" mirror="-1" mirror_dae="False"  front_hind="-1" front_hind_dae="False" />
 </robot>
